File: Remote.sch (EAGLE design)
At the start: 15 parts

Commit message: GND trace width change. Updated silkscreen and created CAM files
Parts:
- U$2: device battery-holders:BLOSSOM-BLM-18650-1PCSNO-SCREWS -> battery-holders-modified:BLOSSOM-BLM-18650-1PCSNO-SCREWS
- renumbered S2 to S1
Changed lines of the file:
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@@
 <part name="JOY" library="SparkFun-Switches" deviceset="JOYSTICK_THUMB" device=""/>
 <part name="FRAME1" library="frames" library_urn="urn:adsk.eagle:library:229" deviceset="A4L-LOC" device=""/>
-<part name="U$2" library="battery-holders" deviceset="BLOSSOM-BLM-18650-1PCS" device="NO-SCREWS" value="BLOSSOM-BLM-18650-1PCSNO-SCREWS"/>
+<part name="U$2" library="battery-holders-modified" deviceset="BLOSSOM-BLM-18650-1PCS" device="NO-SCREWS" value="BLOSSOM-BLM-18650-1PCSNO-SCREWS"/>
 <part name="+3V1" library="supply1" library_urn="urn:adsk.eagle:library:371" deviceset="+3V3" device=""/>
 <part name="GND1" library="supply1" library_urn="urn:adsk.eagle:library:371" deviceset="GND" device=""/>
@@
 <part name="GND2" library="supply1" library_urn="urn:adsk.eagle:library:371" deviceset="GND" device=""/>
 <part name="D1" library="diode" library_urn="urn:adsk.eagle:library:210" deviceset="DIODE-" device="SOD323-W" package3d_urn="urn:adsk.eagle:package:43418/1" value="CUS10S30"/>
-<part name="S2" library="switch-omron" library_urn="urn:adsk.eagle:library:377" deviceset="10-XX" device="" package3d_urn="urn:adsk.eagle:package:27496/1"/>
+<part name="S1" library="switch-omron" library_urn="urn:adsk.eagle:library:377" deviceset="10-XX" device="" package3d_urn="urn:adsk.eagle:package:27496/1"/>
 <part name="GND6" library="supply1" library_urn="urn:adsk.eagle:library:371" deviceset="GND" device=""/>
 <part name="GND7" library="supply1" library_urn="urn:adsk.eagle:library:371" deviceset="GND" device=""/>
@@
 <attribute name="VALUE" x="-66.2686" y="124.46" size="1.778" layer="96" rot="R90"/>
 </instance>
-<instance part="S2" gate="1" x="-30.48" y="106.68" smashed="yes">
+<instance part="S1" gate="1" x="-30.48" y="106.68" smashed="yes">
 <attribute name="NAME" x="-36.83" y="104.14" size="1.778" layer="95" rot="R90"/>
 <attribute name="VALUE" x="-34.29" y="109.855" size="1.778" layer="96" rot="R90"/>
@@
 <wire x1="-10.16" y1="91.44" x2="-10.16" y2="88.9" width="0.1524" layer="91"/>
 <wire x1="-10.16" y1="88.9" x2="-20.32" y2="88.9" width="0.1524" layer="91"/>
-<pinref part="S2" gate="1" pin="P"/>
+<pinref part="S1" gate="1" pin="P"/>
 <wire x1="-30.48" y1="101.6" x2="-30.48" y2="88.9" width="0.1524" layer="91"/>
 <junction x="-30.48" y="88.9"/>
-<pinref part="S2" gate="1" pin="P1"/>
+<pinref part="S1" gate="1" pin="P1"/>
 <wire x1="-27.94" y1="101.6" x2="-30.48" y2="101.6" width="0.1524" layer="91"/>
 <junction x="-30.48" y="101.6"/>
@@
 <net name="N$19" class="0">
 <segment>
-<pinref part="S2" gate="1" pin="S"/>
+<pinref part="S1" gate="1" pin="S"/>
 <wire x1="-30.48" y1="111.76" x2="-30.48" y2="119.38" width="0.1524" layer="91"/>
 <wire x1="-30.48" y1="119.38" x2="12.7" y2="119.38" width="0.1524" layer="91"/>
 <pinref part="ARDUINO-PRO-MINI-3V3" gate="G$1" pin="D4"/>
-<pinref part="S2" gate="1" pin="S1"/>
+<pinref part="S1" gate="1" pin="S1"/>
 <wire x1="-27.94" y1="111.76" x2="-30.48" y2="111.76" width="0.1524" layer="91"/>
 <junction x="-30.48" y="111.76"/>
